File: PCB/SMD/OpenLaserMouse.kicad_pcb (KiCad board)
At the start: 2 copper layers, 56 x 84 mm, 24 parts, among them J1 Amiga_Conn, M1 ADNS-9800, Q1 IRLML6302TRPBF, SW2 LEFT, SW3 RIGHT

Commit message: Adjustments and Photos
Adjusted Mouting Holes on the PCB's
Added Photos of V1.1
Tidy up
Parts:
- moved MHe 0.42 mm to (67.9, 116.5)
- renumbered MH2 to MHe
Changed lines of the file:
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@@
-(kicad_pcb (version 20171130) (host pcbnew "(5.1.0-0)")
+(kicad_pcb (version 20171130) (host pcbnew "(5.1.4-0-10_14)")
   (general
     (thickness 1.6)
@@
     (mod_text_size 1 1)
     (mod_text_width 0.15)
-    (pad_size 3 3)
-    (pad_drill 1.5)
+    (pad_size 6 6)
+    (pad_drill 6)
     (pad_to_mask_clearance 0.051)
     (solder_mask_min_width 0.25)
@@
   )
   (module MountingHole:MountingHole_5.3mm_M5 (layer F.Cu)
-    (at 67.945 116.078)
-    (descr "Mounting Hole 5.3mm, no annular, M5")
-    (tags "mounting hole 5.3mm no annular m5")
-    (attr virtual)
-    (fp_text reference MH2 (at 0 -3.429) (layer F.SilkS) hide
-      (effects (font (size 1 1) (thickness 0.15)))
-    )
-    (fp_text value "Mouse Hole 2" (at 0 3.429) (layer F.Fab) hide
-      (effects (font (size 1 1) (thickness 0.15)))
-    )
-    (fp_text user %R (at 0.3 0) (layer F.Fab) hide
-      (effects (font (size 1 1) (thickness 0.15)))
-    )
-    (pad 1 np_thru_hole circle (at 0 0) (size 5.3 5.3) (drill 5.3) (layers *.Cu *.Mask))
-  )
-  (module MountingHole:MountingHole_5.3mm_M5 (layer F.Cu)
     (at 68.0085 73.9775)
     (descr "Mounting Hole 5.3mm, no annular, M5")
@@
       (effects (font (size 1 1) (thickness 0.15)))
     )
-    (pad 1 np_thru_hole circle (at 0 0) (size 5.3 5.3) (drill 5.3) (layers *.Cu *.Mask))
+    (pad "" np_thru_hole circle (at 0 0) (size 6 6) (drill 6) (layers *.Cu *.Mask))
+  )
+  (module MountingHole:MountingHole_5.3mm_M5 (layer F.Cu)
+    (at 67.945 116.5)
+    (descr "Mounting Hole 5.3mm, no annular, M5")
+    (tags "mounting hole 5.3mm no annular m5")
+    (attr virtual)
+    (fp_text reference MHe (at 0 -3.429) (layer F.SilkS) hide
+      (effects (font (size 1 1) (thickness 0.15)))
+    )
+    (fp_text value "Mouse Hole 2" (at 0 3.429) (layer F.Fab) hide
+      (effects (font (size 1 1) (thickness 0.15)))
+    )
+    (fp_text user %R (at 0.3 0) (layer F.Fab) hide
+      (effects (font (size 1 1) (thickness 0.15)))
+    )
+    (pad "" np_thru_hole circle (at 0 0) (size 6 6) (drill 6) (layers *.Cu *.Mask))
   )
   (module Resistor_SMD:R_0805_2012Metric (layer F.Cu)
