File: PCB/THT/OpenLaserMouseTHT.kicad_pcb (KiCad board)
At the start: 2 copper layers, 56 x 84 mm, 24 parts, among them J1 Amiga_Conn, M1 ADNS-9800, Q1 ZVP2106A, SW2 LEFT, SW3 RIGHT

Commit message: Added ST Mouse PCB
Added ST Mouse PCB
Fixed Wrong Fillplane on Amiga PCB
Parts:
- renumbered MHe to MH2
Routing:
- net GND: track 232.8 -> 18.5 mm
- net Net-(A1-Pad1): vias 7 -> 0
- added copper zone on B.Cu, net GND
- added copper zone on F.Cu, net GND
- removed copper zone on B.Cu, net Net-(A1-Pad1)
- removed copper zone on F.Cu, net Net-(A1-Pad1)
Other:
- board text added: "Open Laser Mouse V1.4 2020 By Chrissy"
- board text removed: "Open Laser Mouse V1.3 2020 By Chrissy"
